Commit message: update configs

File: assets/robots/franka_panda/panda.urdf (robot description, URDF)
Before this commit: robot panda, 13 links, 12 joints
Links:
- link panda_hand: geometry collision mesh filename=package://percept/assets/robots/franka_panda/meshes/collisi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; visual mesh filename=package://percept/assets/robots/franka_panda/meshes/visual/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
- link panda_leftfinger: geometry collision mesh filename=package://percept/assets/robots/franka_panda/meshes/collisi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; visual mesh filename=package://percept/assets/robots/franka_panda/meshes/visual/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
- link panda_link0: geometry collision mesh filename=package://percept/assets/robots/franka_panda/meshes/collisi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; visual mesh filename=package://percept/assets/robots/franka_panda/meshes/collisi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
- link panda_link1: geometry collision mesh filename=package://percept/assets/robots/franka_panda/meshes/collisi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; visual mesh filename=package://percept/assets/robots/franka_panda/meshes/visual/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
- link panda_link2: geometry collision mesh filename=package://percept/assets/robots/franka_panda/meshes/collisi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; visual mesh filename=package://percept/assets/robots/franka_panda/meshes/visual/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
- link panda_link3: geometry collision mesh filename=package://percept/assets/robots/franka_panda/meshes/collisi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; visual mesh filename=package://percept/assets/robots/franka_panda/meshes/visual/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
- link panda_link4: geometry collision mesh filename=package://percept/assets/robots/franka_panda/meshes/collisi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; visual mesh filename=package://percept/assets/robots/franka_panda/meshes/visual/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
- link panda_link5: geometry collision mesh filename=package://percept/assets/robots/franka_panda/meshes/collisi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; visual mesh filename=package://percept/assets/robots/franka_panda/meshes/visual/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
- link panda_link6: geometry collision mesh filename=package://percept/assets/robots/franka_panda/meshes/collisi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; visual mesh filename=package://percept/assets/robots/franka_panda/meshes/visual/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
- link panda_link7: geometry collision mesh filename=package://percept/assets/robots/franka_panda/meshes/collisi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; visual mesh filename=package://percept/assets/robots/franka_panda/meshes/collisi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
- link panda_rightfinger: geometry collision mesh filename=package://percept/assets/robots/franka_panda/meshes/collisi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; visual mesh filename=package://percept/assets/robots/franka_panda/meshes/visual/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

Commit message: add RBS back

File: assets/robots/franka_panda/panda.urdf (robot description, URDF)
Before this commit: robot panda, 13 links, 12 joints
Links:
- link panda_hand: geometry collision mesh filename=package://meshes/collision/hand.obj; visual mesh filename=package://meshes/visual/hand.obj
- link panda_leftfinger: geometry collision mesh filename=package://meshes/collision/finger.obj; visual mesh filename=package://meshes/visual/finger.obj
- link panda_link0: geometry collision mesh filename=package://meshes/collision/link0.obj; visual mesh filename=package://meshes/collision/link0.obj
- link panda_link1: geometry collision mesh filename=package://meshes/collision/link1.obj; visual mesh filename=package://meshes/visual/link1.obj
- link panda_link2: geometry collision mesh filename=package://meshes/collision/link2.obj; visual mesh filename=package://meshes/visual/link2.obj
- link panda_link3: geometry collision mesh filename=package://meshes/collision/link3.obj; visual mesh filename=package://meshes/visual/link3.obj
- link panda_link4: geometry collision mesh filename=package://meshes/collision/link4.obj; visual mesh filename=package://meshes/visual/link4.obj
- link panda_link5: geometry collision mesh filename=package://meshes/collision/link5.obj; visual mesh filename=package://meshes/visual/link5.obj
- link panda_link6: geometry collision mesh filename=package://meshes/collision/link6.obj; visual mesh filename=package://meshes/visual/link6.obj
- link panda_link7: geometry collision mesh filename=package://meshes/collision/link7.obj; visual mesh filename=package://meshes/collision/link7.obj
- link panda_rightfinger: geometry collision mesh filename=package://meshes/collision/finger.obj; visual mesh filename=package://meshes/visual/finger.obj
