Commit message: mod: fix package name and mtl references in panda files

File: src/perception/assets/panda/panda.urdf (robot description, URDF)
Before this commit: robot panda, 13 links, 12 joints
Links:
- link panda_hand: geometry collision mesh filename=package://percept_core/assets/panda/meshes/collision/hand.o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; visual mesh filename=package://percept_core/assets/panda/meshes/visual/hand.obj
- link panda_leftfinger: geometry collision mesh filename=package://percept_core/assets/panda/meshes/collision/finger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; visual mesh filename=package://percept_core/assets/panda/meshes/visual/finger.obj
- link panda_link0: geometry collision mesh filename=package://percept_core/assets/panda/meshes/collision/link0.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; visual mesh filename=package://percept_core/assets/panda/meshes/collision/link0.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
- link panda_link1: geometry collision mesh filename=package://percept_core/assets/panda/meshes/collision/link1.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; visual mesh filename=package://percept_core/assets/panda/meshes/visual/link1.obj
- link panda_link2: geometry collision mesh filename=package://percept_core/assets/panda/meshes/collision/link2.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; visual mesh filename=package://percept_core/assets/panda/meshes/visual/link2.obj
- link panda_link3: geometry collision mesh filename=package://percept_core/assets/panda/meshes/collision/link3.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; visual mesh filename=package://percept_core/assets/panda/meshes/visual/link3.obj
- link panda_link4: geometry collision mesh filename=package://percept_core/assets/panda/meshes/collision/link4.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; visual mesh filename=package://percept_core/assets/panda/meshes/visual/link4.obj
- link panda_link5: geometry collision mesh filename=package://percept_core/assets/panda/meshes/collision/link5.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; visual mesh filename=package://percept_core/assets/panda/meshes/visual/link5.obj
- link panda_link6: geometry collision mesh filename=package://percept_core/assets/panda/meshes/collision/link6.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; visual mesh filename=package://percept_core/assets/panda/meshes/visual/link6.obj
- link panda_link7: geometry collision mesh filename=package://percept_core/assets/panda/meshes/collision/link7.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; visual mesh filename=package://percept_core/assets/panda/meshes/collision/link7.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
- link panda_rightfinger: geometry collision mesh filename=package://percept_core/assets/panda/meshes/collision/finger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; visual mesh filename=package://percept_core/assets/panda/meshes/visual/finger.obj
